Commit message: edits to README

File: urdf/realsense_mount.xacro (robot description, xacro)
@@ -7,5 +7,5 @@
         <geometry>
           <!-- The path to the visual meshes in the package. -->
-          <mesh filename="package://ur5_with_realsesne/meshes/visual/realsense_mount.STL"/>
+          <mesh filename="package://ur5_with_robotiq_gripper_des/meshes/visual/realsense_mount.STL"/>
         </geometry>
       </visual>
@@ -13,5 +13,5 @@
         <geometry>
           <!-- The path to the collision meshes in the package. -->
-          <mesh filename="package://ur5_with_realsesne/meshes/collision/realsense_mount.STL"/>
+          <mesh filename="package://ur5_with_robotiq_gripper_des/meshes/collision/realsense_mount.STL"/>
         </geometry>
       </collision>

File: urdf/ur5_with_robotiq_gripper.xacro (robot description, xacro)
@@ -4,5 +4,5 @@
   <xacro:include filename="$(find ur_description)/urdf/inc/ur5_macro.xacro" />
   <!-- end-effector -->
-  <xacro:include filename="$(find ur5_with_realsesne)/urdf/realsense_mount.xacro" />
+  <xacro:include filename="$(find ur5_with_robotiq_gripper_des)/urdf/realsense_mount.xacro" />
   <xacro:include filename="$(find robotiq_2f_85_gripper_visualization)/urdf/robotiq_arg2f_85_model_macro.xacro" />
   <xacro:include filename="$(find realsense2_description)/urdf/_d415.urdf.xacro" />
